File: SAMD-UPDI-breakaway.kicad_sch (KiCad schematic)
At the start: 13 parts, among them J1 JTAG, J2 FAB-USB-PCB, J3 FTDI Out, J4 FTDI In, J5 UPDI Out, U1 ATSAMD11C14A-SS, U2 MCP1700

Commit message: Outline and Trace files added
Parts:
- J1: value JTAG -> SWD
Changed lines of the file:
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@@
     (in_bom yes) (on_board yes)
     (property "Reference" "J1" (id 0) (at 78.74 91.0082 0))
-    (property "Value" "JTAG" (id 1) (at 78.74 93.3196 0))
+    (property "Value" "SWD" (id 1) (at 78.74 93.3196 0))
     (property "Footprint" "fab:PinHeader_2x02_P2.54mm_Vertical_SMD" (id 2) (at 77.47 96.52 0)
       (effects (font (size 1.27 1.27)) hide)
@@
     )
     (path "/00000000-0000-0000-0000-000061e95181"
-      (reference "J1") (unit 1) (value "JTAG") (footprint "fab:PinHeader_2x02_P2.54mm_Vertical_SMD")
+      (reference "J1") (unit 1) (value "SWD") (footprint "fab:PinHeader_2x02_P2.54mm_Vertical_SMD")
     )
     (path "/00000000-0000-0000-0000-000061ec0501"

Commit message: Replace RST on JTAG header with Vref.  Labels
ATMEL Ice programmer doesn't use RST, but requires that the target microcontroller's VCC be provided for it to sense.  Remove RST from JTAG header, provide VCC instead.
Connections:
- net *RST: no longer J1.3 (Pin_3), U1.6 (PA28/~{RST})
- net +3V3: now also J1.3 (Pin_3)
Changed lines of the file:
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@@
   (junction (at 187.96 99.06) (diameter 0) (color 0 0 0 0)
   )
+  (junction (at 90.17 73.66) (diameter 0) (color 0 0 0 0)
+  )
   (junction (at 187.96 104.14) (diameter 0) (color 0 0 0 0)
   )
@@
     (stroke (width 0) (type default) (color 0 0 0 0))
   )
+  (wire (pts (xy 69.85 99.06) (xy 69.85 73.66))
+    (stroke (width 0) (type default) (color 0 0 0 0))
+  )
   (wire (pts (xy 170.18 109.22) (xy 170.18 104.14))
     (stroke (width 0) (type default) (color 0 0 0 0))
@@
     (stroke (width 0) (type default) (color 0 0 0 0))
   )
-  (wire (pts (xy 93.98 91.44) (xy 92.71 91.44))
-    (stroke (width 0) (type default) (color 0 0 0 0))
-  )
   (wire (pts (xy 160.02 73.66) (xy 166.37 73.66))
     (stroke (width 0) (type default) (color 0 0 0 0))
@@
     (stroke (width 0) (type default) (color 0 0 0 0))
   )
+  (wire (pts (xy 106.68 81.28) (xy 106.68 73.66))
+    (stroke (width 0) (type default) (color 0 0 0 0))
+  )
   (wire (pts (xy 166.37 73.66) (xy 166.37 76.2))
     (stroke (width 0) (type default) (color 0 0 0 0))
@@
     (stroke (width 0) (type default) (color 0 0 0 0))
   )
+  (wire (pts (xy 106.68 73.66) (xy 90.17 73.66))
+    (stroke (width 0) (type default) (color 0 0 0 0))
+  )
   (wire (pts (xy 127 106.68) (xy 119.38 106.68))
     (stroke (width 0) (type default) (color 0 0 0 0))
@@
     (stroke (width 0) (type default) (color 0 0 0 0))
   )
+  (wire (pts (xy 69.85 73.66) (xy 90.17 73.66))
+    (stroke (width 0) (type default) (color 0 0 0 0))
+  )
   (wire (pts (xy 119.38 93.98) (xy 134.62 93.98))
     (stroke (width 0) (type default) (color 0 0 0 0))
@@
     (stroke (width 0) (type default) (color 0 0 0 0))
   )
-  (wire (pts (xy 92.71 85.09) (xy 69.85 85.09))
-    (stroke (width 0) (type default) (color 0 0 0 0))
-  )
   (wire (pts (xy 170.18 99.06) (xy 152.4 99.06))
     (stroke (width 0) (type default) (color 0 0 0 0))
@@
   )
   (wire (pts (xy 152.4 93.98) (xy 187.96 93.98))
-    (stroke (width 0) (type default) (color 0 0 0 0))
-  )
-  (wire (pts (xy 92.71 91.44) (xy 92.71 85.09))
-    (stroke (width 0) (type default) (color 0 0 0 0))
-  )
-  (wire (pts (xy 69.85 85.09) (xy 69.85 99.06))
     (stroke (width 0) (type default) (color 0 0 0 0))
   )
@@
     (in_bom yes) (on_board yes)
     (property "Reference" "U1" (id 0) (at 93.98 78.74 0))
-    (property "Value" "ATSAMD11C14A-SS" (id 1) (at 93.98 81.28 0))
+    (property "Value" "ATSAMD11C14A-SS" (id 1) (at 119.38 81.28 0))
     (property "Footprint" "fab:SOIC-14_3.9x8.7mm_P1.27mm" (id 2) (at 106.68 125.73 0)
       (effects (font (size 1.27 1.27)) hide)
@@
     (pin "9")
   )
-  (symbol (lib_id "power:+3.3V") (at 106.68 81.28 0) (unit 1)
+  (symbol (lib_id "power:+3.3V") (at 90.17 73.66 0) (unit 1)
     (in_bom yes) (on_board yes)
-    (property "Reference" "#PWR0107" (id 0) (at 106.68 85.09 0)
-      (effects (font (size 1.27 1.27)) hide)
-    )
-    (property "Value" "+3.3V" (id 1) (at 107.061 76.8858 0))
-    (property "Footprint" "" (id 2) (at 106.68 81.28 0)
-      (effects (font (size 1.27 1.27)) hide)
-    )
-    (property "Datasheet" "" (id 3) (at 106.68 81.28 0)
-      (effects (font (size 1.27 1.27)) hide)
-    )
+    (property "Reference" "#PWR0107" (id 0) (at 90.17 77.47 0)
+      (effects (font (size 1.27 1.27)) hide)
+    )
+    (property "Value" "+3.3V" (id 1) (at 90.551 69.2658 0))
+    (property "Footprint" "" (id 2) (at 90.17 73.66 0)
+      (effects (font (size 1.27 1.27)) hide)
+    )
+    (property "Datasheet" "" (id 3) (at 90.17 73.66 0)
+      (effects (font (size 1.27 1.27)) hide)
+    )
