File: Blinkenlights-version/SAMD-UPDI-breakaway-blinkenlights.kicad_pcb (KiCad board)
At the start: 2 copper layers, 79.1 x 17 mm, 17 parts, among them J1 SWD, J2 FAB-USB-PCB, J3 FTDI Out, J4 FTDI In, J5 UPDI Out, U1 ATSAMD11C14A-SS, U2 MCP1700

Commit message: Updated Blinkenlights readme
Parts:
- D1: value LED -> RED LED
- D2: value LED -> GRN LED
- R6: value 1.2K -> 500
Changed lines of the file:
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@@
       (effects (font (size 1 1) (thickness 0.15)))
     )
-    (fp_text value "1.2K" (at 0 1.9 90) (layer "F.Fab")
+    (fp_text value "500" (at 0 -1.7 90) (layer "F.Fab")
       (effects (font (size 1 1) (thickness 0.15)))
     )
@@
       (effects (font (size 1 1) (thickness 0.15)))
     )
-    (fp_text value "LED" (at 0 1.9 90) (layer "F.Fab")
+    (fp_text value "GRN LED" (at 0 1.9 90) (layer "F.Fab")
       (effects (font (size 1 1) (thickness 0.15)))
     )
@@
       (effects (font (size 1 1) (thickness 0.15)))
     )
-    (fp_text value "LED" (at 0 1.9 90) (layer "F.Fab")
+    (fp_text value "RED LED" (at 0 1.9 90) (layer "F.Fab")
       (effects (font (size 1 1) (thickness 0.15)))
     )
